Commit message: 7.16

File: bittle_rl_gym/assets/urdf/bittle_PRD_v2.urdf (robot description, URDF)
Before this commit: robot bittle, 17 links, 16 joints
Links:
- link base-frame-link: geometry collision mesh filename=bittle_rl_gym/assets/meshes/base_frame.001.obj scale=0.1 0.1 0.1; visual mesh filename=bittle_rl_gym/assets/meshes/base_frame.obj scale=0.1 0.1 0.1
- link battery-link: geometry collision mesh filename=bittle_rl_gym/assets/meshes/battery.001.obj scale=0.1 0.1 0.1; visual mesh filename=bittle_rl_gym/assets/meshes/battery.obj scale=0.1 0.1 0.1
- link cover-link: geometry collision mesh filename=bittle_rl_gym/assets/meshes/cover.001.obj scale=0.1 0.1 0.1; visual mesh filename=bittle_rl_gym/assets/meshes/cover.obj scale=0.1 0.1 0.1
- link imu_link: geometry visual mesh filename=bittle_rl_gym/assets/meshes/Cube.011.obj scale=0.002474 0.002474 0.000635
- link left-back-knee-link: geometry collision mesh filename=bittle_rl_gym/assets/meshes/left_knee.002.obj scale=0.1 0.1 0.1; visual mesh filename=bittle_rl_gym/assets/meshes/left_knee.001.obj scale=0.1 0.1 0.1
- link left-back-shoulder-link: geometry collision mesh filename=bittle_rl_gym/assets/meshes/shoulder.004.obj scale=0.1 0.1 0.1; visual mesh filename=bittle_rl_gym/assets/meshes/shoulder.001.obj scale=0.1 0.1 0.1
- link left-front-knee-link: geometry collision mesh filename=bittle_rl_gym/assets/meshes/left_knee.003.obj scale=0.1 0.1 0.1; visual mesh filename=bittle_rl_gym/assets/meshes/left_knee.obj scale=0.1 0.1 0.1
- link left-front-shoulder-link: geometry collision mesh filename=bittle_rl_gym/assets/meshes/shoulder.007.obj scale=0.1 0.1 0.1; visual mesh filename=bittle_rl_gym/assets/meshes/shoulder.obj scale=0.1 0.1 0.1
- link mainboard_link: geometry visual mesh filename=bittle_rl_gym/assets/meshes/Plane.obj scale=0.027649 0.028815 0.025599
- link right-back-knee-link: geometry collision mesh filename=bittle_rl_gym/assets/meshes/right_knee.002.obj scale=0.1 0.1 0.1; visual mesh filename=bittle_rl_gym/assets/meshes/right_knee.001.obj scale=0.1 0.1 0.1
- link right-back-shoulder-link: geometry collision mesh filename=bittle_rl_gym/assets/meshes/shoulder.005.obj scale=0.1 0.1 0.1; visual mesh filename=bittle_rl_gym/assets/meshes/shoulder.002.obj scale=0.1 0.1 0.1
- link right-front-knee-link: geometry collision mesh filename=bittle_rl_gym/assets/meshes/right_knee.003.obj scale=0.1 0.1 0.1; visual mesh filename=bittle_rl_gym/assets/meshes/right_knee.obj scale=0.1 0.1 0.1
- link right-front-shoulder-link: geometry collision mesh filename=bittle_rl_gym/assets/meshes/shoulder.006.obj scale=0.1 0.1 0.1; visual mesh filename=bittle_rl_gym/assets/meshes/shoulder.003.obj scale=0.1 0.1 0.1

Commit message: 7.17: periodical reward composition + sim_params + rewards + PD

File: bittle_rl_gym/assets/urdf/bittle_PRD_v2.urdf (robot description, URDF)
Before this commit: robot bittle, 17 links, 16 joints
Links:
- link base-frame-link: geometry collision mesh filename=../meshes/base_frame.001.obj scale=0.1 0.1 0.1; visual mesh filename=../meshes/base_frame.obj scale=0.1 0.1 0.1
- link battery-link: geometry collision mesh filename=../meshes/battery.001.obj scale=0.1 0.1 0.1; visual mesh filename=../meshes/battery.obj scale=0.1 0.1 0.1
- link cover-link: geometry collision mesh filename=../meshes/cover.001.obj scale=0.1 0.1 0.1; visual mesh filename=../meshes/cover.obj scale=0.1 0.1 0.1
- link imu_link: geometry visual mesh filename=../meshes/Cube.011.obj scale=0.002474 0.002474 0.000635
- link left-back-knee-link: geometry collision mesh filename=../meshes/left_knee.002.obj scale=0.1 0.1 0.1; visual mesh filename=../meshes/left_knee.001.obj scale=0.1 0.1 0.1
- link left-back-shoulder-link: geometry collision mesh filename=../meshes/shoulder.004.obj scale=0.1 0.1 0.1; visual mesh filename=../meshes/shoulder.001.obj scale=0.1 0.1 0.1
- link left-front-knee-link: geometry collision mesh filename=../meshes/left_knee.003.obj scale=0.1 0.1 0.1; visual mesh filename=../meshes/left_knee.obj scale=0.1 0.1 0.1
- link left-front-shoulder-link: geometry collision mesh filename=../meshes/shoulder.007.obj scale=0.1 0.1 0.1; visual mesh filename=../meshes/shoulder.obj scale=0.1 0.1 0.1
- link mainboard_link: geometry visual mesh filename=../meshes/Plane.obj scale=0.027649 0.028815 0.025599
- link right-back-knee-link: geometry collision mesh filename=../meshes/right_knee.002.obj scale=0.1 0.1 0.1; visual mesh filename=../meshes/right_knee.001.obj scale=0.1 0.1 0.1
- link right-back-shoulder-link: geometry collision mesh filename=../meshes/shoulder.005.obj scale=0.1 0.1 0.1; visual mesh filename=../meshes/shoulder.002.obj scale=0.1 0.1 0.1
- link right-front-knee-link: geometry collision mesh filename=../meshes/right_knee.003.obj scale=0.1 0.1 0.1; visual mesh filename=../meshes/right_knee.obj scale=0.1 0.1 0.1
- link right-front-shoulder-link: geometry collision mesh filename=../meshes/shoulder.006.obj scale=0.1 0.1 0.1; visual mesh filename=../meshes/shoulder.003.obj scale=0.1 0.1 0.1
