Commit message: 8.22: Add foot periodicity

File: bittle_rl_gym/assets/bittle-official/urdf/Bittle_Petoi.urdf (robot description, URDF)
Before this commit: robot bittle, 87 links, 86 joints
Links:
- added link lf-foot-sole-link; visual sphere radius=0.001
- added link lr-foot-sole-link; visual sphere radius=0.001
- added link rf-foot-sole-link; visual sphere radius=0.001
- added link rr-foot-sole-link; visual sphere radius=0.001
Joints:
- added joint lf-foot-sole-joint: type fixed, parent shank_lf_1, child lf-foot-sole-link, origin xyz=0.05 -0.005 0 rpy=0 0 0
- added joint lr-foot-sole-joint: type fixed, parent shank_lr_1, child lr-foot-sole-link, origin xyz=0.05 -0.005 0 rpy=0 0 0
- added joint rf-foot-sole-joint: type fixed, parent shank_rf_1, child rf-foot-sole-link, origin xyz=0.05 0.005 0 rpy=0 0 0
- added joint rr-foot-sole-joint: type fixed, parent shank_rr_1, child rr-foot-sole-link, origin xyz=0.05 0.005 0 rpy=0 0 0
